Commit message: diff-drive-pontoon: may need to refine PID

File: usv_vrx/usv_description/configs/default_config.urdf (robot description, URDF)
Before this commit: robot WAM-V, 23 links, 22 joints
Links:
- added link lateral_engine_link, mass 15; collision box size=0.12 0.15 0.12; collision box size=0.2 0.15 0.83
- added link lateral_propeller_link, mass 0.5; collision cylinder length=0.18 radius=0.24; visual mesh filename=package://wamv_description/models/propeller/mesh/propeller.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
Joints:
- added joint lateral_chasis_engine_joint: type revolute, parent base_link, child lateral_engine_link, origin xyz=1.186888 0.300000 0.318237 rpy=0.0 0.0 1.570796327, axis 0 0 1, limit lower=-3.14159265359 upper=3.14159265359 effort=10 velocity=10
- added joint lateral_engine_propeller_joint: type continuous, parent lateral_engine_link, child lateral_propeller_link, origin xyz=-0.278156 0 -0.509371 rpy=0 0 0, axis 1 0 0, limit effort=100 velocity=100
