Commit message: ekflocalization is back!

File: usv_vrx/usv_description/configs/usv_mtu.urdf (robot description, URDF)
Before this commit: robot WAM-V, 22 links, 21 joints
Links:
- removed link lateral_engine_link
- removed link lateral_propeller_link
Joints:
- removed joint lateral_chasis_engine_joint
- removed joint lateral_engine_propeller_joint
- joint lidar_wamv_post_arm_to_lidar_wamv_joint: origin xyz=0.04 0 0.05 rpy=0.0 0.0 0.0 -> xyz=0.04 0 0.7 rpy=0.0 0 0.0

Commit message: Initial commit of vrx_ws

File: usv_vrx/usv_description/configs/usv_mtu.urdf (robot description, URDF)
Before this commit: robot WAM-V, 22 links, 21 joints
Links:
- link front_mid_camera_link: geometry collision box size=0.036 0.03 0.03; collision cylinder length=0.042 radius=0.015
Joints:
- joint front_mid_camera_to_front_mid_camera_link_optical_joint: origin xyz=0 0 0 rpy=-1.5707963267948966 0 -1.5707963267948966 -> xyz=0 0 0 rpy=0 -1.57 -1.57

File: vrx/vrx_2019/worlds/example_course.world.xacro (robot description, xacro)
@@ -43,9 +43,9 @@
       <uri>model://simple_maze</uri>
       <pose>20.652985 14.555411 0 0 0 0.190745</pose>
-    </include>-->
+    </include>
     <include>
       <uri>model://onepath_maze</uri>
       <pose>-35.5535 64.792 0 0 0 -1.42</pose>
-    </include>
+    </include>-->
     <xacro:include filename="$(find vrx_gazebo)/worlds/xacros/usv_wind_plugin.xacro"/>
     <xacro:usv_wind_gazebo>

File: vrx/wave_gazebo/world_models/ocean_waves/model.xacro (robot description, xacro)
@@ -16,6 +16,6 @@
   Modified to include wave field model and visual plugins.
 -->
-<world xmlns:xacro="http://ros.org/wiki/xacro"> <!-- period cannot be zero -->
-  <xacro:macro name="ocean_waves" params="gain:=0.0 period:=0.01
+<world xmlns:xacro="http://ros.org/wiki/xacro">
+  <xacro:macro name="ocean_waves" params="gain:=0.1 period:=5
                      direction_x:=1.0 direction_y:=0.0
                      angle:=0.4 scale:=1.5">
